File: eagle/BeagleQ-v02.brd (EAGLE design)
At the start: 100 x 80 mm, 23 parts, among them IC2 AT24CP, Q1 TIP120

Commit message: Functioning hardware
Parts:
- removed SG1: F/CM12P, buzzer:F/CM12P
- removed VDD_12V: (no value), pinhead:1X02/90
- added D2: 1N4004, adafruit:DO41-10
- added J1, J2, J3: DCJ0202, houseofbeck:DCJ0202
- added JP5: RCA, SparkFun-Connectors:RCA
- added P1: (no value), jst-ph:JST-PH4
- added SP1: SPEAKER/PS12, adafruit:PS12
- JP2: device pinhead:1X04/90 -> SparkFun-Connectors:1X04
- R10, R11, R8, R9: value 22k -> 10k
- SV2: device pinhead:1X08/90 -> jumper:JP5Q
- moved JP2 57.5 mm to (67.3, 31.8)
- moved SV2 15.5 mm to (25.4, 49.5)
- moved R1 13.4 mm to (36.2, 44.5)
- moved R10 13.4 mm to (36.2, 49.5)
- moved R11 13.4 mm to (36.2, 47.0)
- moved R8 13.4 mm to (36.2, 54.6)
- moved R9 13.4 mm to (36.2, 52.1)
- moved LED1 11.4 mm to (45.7, 45.1)
- moved JP1 8.54 mm to (60.3, 36.8)
- moved C1 7.24 mm to (65.4, 55.2), turned to 90 degrees
- moved Q1 4.49 mm to (29.8, 36.2)
- moved R7 3.81 mm to (62.2, 52.1)
- moved R2 0.63 mm to (43.2, 22.2)
- moved R4 0.63 mm to (43.2, 28.6)
Connections:
- new net EHRPWM2A: LED1.K, R1.2, U$1.19
- net AIN1: now also J1.2, SV2.9; no longer SV2.7
- net AIN2: now also J2.2, SV2.7; no longer SV2.6
- net AIN3: now also J3.2
- net AIN4: now also SV2.3; no longer SV2.4
- net BLOWER_H: now also D2.C, JP5.PIN, P1.3; no longer VDD_12V.1
- net BLOWER_L: now also D2.A, JP5.SHELL
- net EHRPWM1A: no longer LED1.K, R1.2
- net EHRPWM1B: now also SP1.P$1; no longer SG1.+
- net GND: now also JP2.2, P1.1, P1.4, SP1.P$2; no longer JP2.4, SG1.-, VDD_12V.2
- net GNDA_ADC: now also J1.1, J1.3, J2.1, J2.3, J3.1, J3.3, SV2.10, SV2.4, SV2.6
- net I2C2_SCL: now also JP2.4; no longer JP2.2
- net VDD: now also P1.2
Routing:
- net BLOWER_H: track 7.19 -> 72.7 mm
- net GNDA_ADC: track 21.5 -> 70.7 mm
- net I2C2_SCL: track 105.3 -> 61.3 mm
- net EHRPWM1A: track 42.0 -> 0.00 mm
- net VDD: track 76.9 -> 36.2 mm
- net I2C2_SDA: track 102.0 -> 66.1 mm
- net BLOWER_L: track 7.18 -> 42.5 mm
- net EHRPWM2A: track 0.00 -> 34.8 mm
- net AIN3: track 21.4 -> 36.8 mm
- net AIN2: track 21.4 -> 29.3 mm
- net AIN4: track 28.5 -> 22.5 mm
- net N$3: track 7.18 -> 13.0 mm
- net AIN1: track 15.2 -> 20.7 mm
- net N$5: track 14.0 -> 8.48 mm
- net EHRPWM1B: track 12.6 -> 7.85 mm
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Other:
- board text added: "BeagleQ V2.1"
- board text added: "FAN"
- board text added: "FOOD1"
- board text added: "FOOD2"
- board text added: "PIT"
- board text removed: "2"
- board text removed: "3"
- board text removed: "4"
- board text removed: "BeagleQ V2.0"
