File: eagle/BeagleQ-v02.sch (EAGLE design)
At the start: 23 parts, among them IC2 AT24CP, Q1 TIP120

Commit message: Functioning hardware
Parts:
- removed SG1: F/CM12P, buzzer:F/CM12P
- removed VDD_12V: (no value), pinhead:PINHD-1X2/90
- added D2: 1N4004, adafruit:1N4004
- added J1, J2, J3: DCJ0202, houseofbeck:DCJ0202
- added JP5: RCA, SparkFun-Connectors:RCA
- added P1: (no value), jst-ph:JST-PH4
- added SP1: SPEAKER/PS12, adafruit:SPEAKER/PS12
- JP2: device pinhead:PINHD-1X4/90 -> SparkFun-Connectors:M04PTH
- R10, R11, R8, R9: value 22k -> 10k
- SV2: device pinhead:PINHD-1X8/90 -> jumper:JP5Q
Connections:
- new net EHRPWM2A: LED1.C, R1.2, U$1.EHRPWM2A
- net AIN1: now also J1.2, SV2.9; no longer SV2.7
- net AIN2: now also J2.2, SV2.7; no longer SV2.6
- net AIN3: now also J3.2
- net AIN4: now also SV2.3; no longer SV2.4
- net BLOWER_H: now also D2.C, JP5.PIN, P1.3; no longer VDD_12V.1
- net BLOWER_L: now also D2.A, JP5.SHELL
- net EHRPWM1A: no longer LED1.C, R1.2
- net EHRPWM1B: now also SP1.+; no longer SG1.1
- net GND: now also JP2.2, P1.1, P1.4, SP1.-; no longer JP2.4, SG1.2, VDD_12V.2
- net GNDA_ADC: now also J1.1, J1.3, J2.1, J2.3, J3.1, J3.3, SV2.10, SV2.4, SV2.6
- net I2C2_SCL: now also JP2.4; no longer JP2.2
- net VDD: now also P1.2
